File: Kicad Defi/Defi.kicad_sch (KiCad schematic)
At the start: 37 parts, among them J1 Omnimate2, J10 Autocom4, J2 Autocom2, J3 Autocom2, J4 Autocom4, J4 Mounting_Screw_3mm, J5 Mounting_Screw_3mm, J6 Mounting_Screw_3mm, J8 Autocom4, Q1 IRL510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

Commit message: Mutex + LCD+ENCODEUR+MPU = test validé
Connections:
- net +12P: no longer Q1.3 (S), SW1.2
- net GND: now also Q1.3 (S), SW1.2
